File: dabao_v3c.kicad_pcb (KiCad board)
At the start: 2 copper layers, 21 x 41 mm, 51 parts, among them J1 USB_C_Receptacle_USB2.0_16P, SW1 SW_Push, SW2 SW_Push, U1 baochip1x, U3 Baochip, U4 MT3406, U5 EMS4000RSW, U6 MT3406, Y2 48.000MHz

Commit message: update to production release files
add CE/CS logos
Parts:
- added REF**: Crowd_Supply_Icon_Silk_10mm, Crowd_Supply:Crowd_Supply_Icon_Silk_10mm, B.Cu at (132.2, 87.1)
- added REF**: CE-Logo_8.5x6mm_SilkScreen, Symbol:CE-Logo_8.5x6mm_SilkScreen, B.Cu at (132.3, 75.7)
- C1, C10: value 12pF C0G -> 33pF C0G
Other:
- board text added: "v3e 02/26"
- board text removed: "v3c 11/25"
